File: kicad/file5ACC9B8E.sch (KiCad schematic (older format))
At the start: 24 parts

Commit message: extra push
Parts:
- removed C? (x2): 100µ, symbol C_Small
- removed C?: 10µ, symbol C_Small
- removed C? (x4): 100n, symbol C_Small
- removed D?: D_Zener_Small, symbol D_Zener_Small
- removed D?: 30V, symbol D_Zener_Small
- removed F?: 10AT, symbol Fuse
- removed J?: Conn_01x02, symbol Conn_01x02
- removed Q? (x2): IRF4905, TO_SOT_Packages_THT:TO-220_Vertical, symbol IRF4905
- removed Q? (x3): BC817, TO_SOT_Packages_SMD:SOT-23, symbol BC817
- removed R? (x3): R_Small, symbol R_Small
- removed R?: 2k2, symbol R_Small
- removed R? (x2): 10k, symbol R_Small
- removed R?: 100k, symbol R_Small
- removed U?: ACS725xMATR-20AB, Package_SO:SOIC-16W_7.5x10.3mm_P1.27mm, symbol ACS725xMATR-20AB
Connections:
- no-connect marks 2 -> 0
